Commit message: Fix: Add URDF rotation matrix compatibility check and improve error handling
- Added pre-check for Pinocchio rotation matrix issues in w10.urdf
- Fixed RGBA color values in w10.urdf (125 -> 0.49)
- Added link_tcp end-effector to w10.urdf
- Documented URDF compatibility issues
- Note: w10.urdf still has internal Pinocchio rotation matrix assertion failures
  that require fixing the URDF file or regenerating from SolidWorks

File: src/w10_sim/urdf/w10.urdf (robot description, URDF)
Before this commit: robot w10_sim, 8 links, 7 joints
Links:
- added link link_tcp, mass 0.001
Joints:
- added joint tcp_joint: type fixed, parent Link8, child link_tcp, origin xyz=0 0 0.05 rpy=0 0 0

Commit message: Remove outdated URDF files and add new URDF model for w10 robot. Include new mesh for Link1 and update joint configurations for improved accuracy in simulation.

File: src/w10_sim/urdf/w10.urdf (robot description, URDF)
Before this commit: robot w10_sim, 9 links, 8 joints
Links:
- removed link link_tcp
Joints:
- removed joint tcp_joint
- joint joint3: origin xyz=0 0 0.085 rpy=0 0 0 -> xyz=0 0 0.085 rpy=-1.5708 0 -1.5708
- joint joint4: axis 0 0 -1 -> 0 0 1; origin xyz=0 -0.2815 8.9457E-05 rpy=0 0 0 -> xyz=0 -0.2815 8.9457E-05 rpy=1.5708 0 0
- joint joint5: origin xyz=0.050005 -8.944E-05 0.1435 rpy=0 0 0 -> xyz=0.050005 -8.944E-05 0.1435 rpy=-1.5708 0 0
- joint joint6: origin xyz=-0.049995 -0.1105 1.2129E-05 rpy=0 0 0 -> xyz=-0.049995 -0.1105 1.2129E-05 rpy=1.5708 0 0
- joint joint7: origin xyz=0 -0.062949 0.3162 rpy=0 0 0 -> xyz=0 -0.062949 0.3162 rpy=-1.5708 0 0
- joint joint8: axis 0 0 -1 -> 0 0 1; origin xyz=0 -0.0684 0.062 rpy=0 0 0 -> xyz=0 -0.0684 0.062 rpy=1.5708 0 0
