Commit message: 更新w10new.urdf文件，调整关节限制参数以提高运动范围和精度

File: src/w10_sim/urdf/w10new.urdf (robot description, URDF)
Before this commit: robot w10new, 8 links, 7 joints
Joints:
- joint Joint1: limit lower=0 upper=0 effort=0 velocity=0 -> lower=-3.14159 upper=3.14159 effort=150 velocity=1.57
- joint Joint2: limit lower=0 upper=0 effort=0 velocity=0 -> lower=-3.14159 upper=3.14159 effort=150 velocity=1.57
- joint Joint3: limit lower=0 upper=0 effort=0 velocity=0 -> lower=-3.14159 upper=3.14159 effort=150 velocity=1.57
- joint Joint4: limit lower=0 upper=0 effort=0 velocity=0 -> lower=-3.14159 upper=3.14159 effort=150 velocity=1.57
- joint Joint5: limit lower=0 upper=0 effort=0 velocity=0 -> lower=-3.14159 upper=3.14159 effort=150 velocity=1.57
- joint Joint6: limit lower=0 upper=0 effort=0 velocity=0 -> lower=-3.14159 upper=3.14159 effort=150 velocity=1.57
- joint Joint7: limit lower=0 upper=0 effort=0 velocity=0 -> lower=-3.14159 upper=3.14159 effort=150 velocity=1.57

Commit message: 更新w10new.urdf文件，修正Joint6的位移参数以确保正确的关节位置

File: src/w10_sim/urdf/w10new.urdf (robot description, URDF)
Before this commit: robot w10new, 8 links, 7 joints
Joints:
- joint Joint6: origin xyz=0 -0.000937 0 rpy=1.5708 0 -3.1416 -> xyz=0 0 0 rpy=1.5708 0 -3.1416
