Commit message: 删除多余数据，catsvi改为增量式

File: install/marvin_sim/share/marvin_sim/urdf/7_pendulum.urdf (robot description, URDF)
Before this commit: robot planar_3r_pendulum, 10 links, 9 joints
Links:
- removed link link7
- added link Link7, mass 0.5; collision cylinder length=1.0 radius=0.02; visual cylinder length=1.0 radius=0.02
Joints:
- joint joint7: child link7 -> Link7
- joint joint_tcp: parent link7 -> Link7
